Commit message: Restore LIMB simulation and add GUI sensor recording
- Fix arm reset, joint limits, and interactive controls; restore the Control Center tabs.
- Add BLE, serial, and camera recording tools and Motion AI.
- Add guided labeled BLE capture with old-format CSV output and packet-loss checks.

File: src/simulation/sim/arm/right_arm.urdf (robot description, URDF)
Before this commit: robot right_arm_final, 27 links, 26 joints
Links:
- removed link right_elbow_roty
- removed link right_shoulder_rotx
- removed link right_wrist_rotx
- added link right_shoulder_roty, mass 0.6; collision mesh filename=arm/r_shoulder.stl scale=0.001 0.001 0.001; visual mesh filename=arm/r_shoulder.stl scale=0.001 0.001 0.001
- added link right_wrist_rotation, mass 0.1
- link arm_base_rotated: mass 0.001 -> 0.8; geometry collision mesh filename=arm/r_shoulder_base.stl scale=0.001 0.001 0.001; visual mesh filename=arm/r_shoulder_base.stl scale=0.001 0.001 0.001
- link right_shoulder_rotz: geometry 
- link right_upper_arm: geometry collision mesh filename=arm/bicep.stl scale=0.001 0.001 0.001; visual mesh filename=arm/bicep.stl scale=0.001 0.001 0.001
Joints:
- removed joint jRightElbow_rotz
- removed joint jRightWrist_rotx
- removed joint jRightWrist_rotz
- added joint jRightWrist_rotation: type revolute, parent right_forearm, child right_wrist_rotation, origin xyz=0.310 0.0085 -0.005 rpy=0 0 0, axis 1 0 0, limit lower=0 upper=2.443461 effort=4 velocity=1.745329
- added joint right_hand_mount: type fixed, parent right_wrist_rotation, child right_hand, origin xyz=0 0 -0.006 rpy=0 0 0
- joint jRightElbow_roty: child right_elbow_roty -> right_forearm; limit lower=-1.047198 upper=0 effort=200 velocity=0.698132 -> lower=-1.047198 upper=0 effort=10 velocity=0.698132; origin xyz=0.305 0 0 rpy=0 0 0 -> xyz=0.189 0 0 rpy=0 0 0
- joint jRightShoulder_rotx: child right_shoulder_rotx -> right_upper_arm; limit lower=-1.047198 upper=1.047198 effort=200 velocity=0.698132 -> lower=-1.047198 upper=1.047198 effort=15 velocity=0.698132; origin xyz=0 0 0 rpy=0 0 0 -> xyz=0.116 0 0 rpy=0 0 0; parent right_shoulder_rotz -> right_shoulder_roty
- joint jRightShoulder_roty: child right_upper_arm -> right_shoulder_roty; limit lower=0 upper=1.570796 effort=200 velocity=0.349066 -> lower=0 upper=1.570796 effort=20 velocity=0.349066; parent right_shoulder_rotx -> right_shoulder_rotz
- joint jRightShoulder_rotz: limit lower=-0.698132 upper=-0.087266 effort=200 velocity=0.349066 -> lower=-0.698132 upper=-0.087266 effort=20 velocity=0.349066
