Commit message: sim fix?
.

File: src/simulation/sim/arm/left_arm.urdf (robot description, URDF)
Before this commit: robot left_arm_final, 27 links, 26 joints
Links:
- link arm_base_rotated: mass None -> 0.001
- link base_link: mass None -> 0.001
- link hand_cover_link: mass None -> 0.05
Joints:
- joint jLeftElbow_roty: limit lower=-3.14 upper=3.14 effort=200 velocity=100.0 -> lower=0 upper=1.047198 effort=200 velocity=0.698132
- joint jLeftElbow_rotz: limit lower=-3.14 upper=3.14 effort=200 velocity=100.0 -> lower=0 upper=2.443461 effort=200 velocity=1.745329
- joint jLeftShoulder_rotx: limit lower=-3.14 upper=3.14 effort=200 velocity=100.0 -> lower=-1.047198 upper=1.047198 effort=200 velocity=0.698132
- joint jLeftShoulder_roty: limit lower=-3.14 upper=3.14 effort=200 velocity=100.0 -> lower=0 upper=1.570796 effort=200 velocity=0.349066
- joint jLeftShoulder_rotz: limit lower=-3.14 upper=3.14 effort=200 velocity=100.0 -> lower=-0.698132 upper=-0.087266 effort=200 velocity=0.349066
- joint jLeftWrist_rotx: axis -1 0 0 -> (none); limit lower=-3.14 upper=3.14 effort=200 velocity=100.0 -> (none); type revolute -> fixed
- joint jLeftWrist_rotz: axis 0 0 -1 -> (none); limit lower=-3.14 upper=3.14 effort=200 velocity=100.0 -> (none); type revolute -> fixed

File: src/simulation/sim/arm/right_arm.urdf (robot description, URDF)
Before this commit: robot right_arm_final, 27 links, 26 joints
Links:
- link arm_base_rotated: mass None -> 0.001
- link base_link: mass None -> 0.001
- link hand_cover_link: mass None -> 0.05
- link right_elbow_roty: mass 1.0 -> 0.1; geometry visual sphere radius=0.02
- link right_forearm: mass 0.1 -> 1.0; geometry collision mesh filename=arm/r_forearm.stl scale=0.001 0.001 0.001; visual mesh filename=arm/r_forearm.stl scale=0.001 0.001 0.001
- link right_hand: mass 0.1 -> 0.4; geometry collision mesh filename=arm/r_hand.stl scale=0.001 0.001 0.001; visual mesh filename=arm/r_hand.stl scale=0.001 0.001 0.001
- link right_wrist_rotx: mass 0.4 -> 0.1; geometry visual sphere radius=0.02
Joints:
- joint jRightElbow_roty: limit lower=-3.14 upper=3.14 effort=200 velocity=100.0 -> lower=-1.047198 upper=0 effort=200 velocity=0.698132
- joint jRightElbow_rotz: limit lower=-3.14 upper=3.14 effort=200 velocity=100.0 -> lower=0 upper=2.443461 effort=200 velocity=1.745329
- joint jRightShoulder_rotx: limit lower=-3.14 upper=3.14 effort=200 velocity=100.0 -> lower=-1.047198 upper=1.047198 effort=200 velocity=0.698132
- joint jRightShoulder_roty: limit lower=-3.14 upper=3.14 effort=200 velocity=100.0 -> lower=0 upper=1.570796 effort=200 velocity=0.349066
- joint jRightShoulder_rotz: limit lower=-3.14 upper=3.14 effort=200 velocity=100.0 -> lower=-0.698132 upper=-0.087266 effort=200 velocity=0.349066
- joint jRightWrist_rotx: axis 1 0 0 -> (none); limit lower=-3.14 upper=3.14 effort=200 velocity=100.0 -> (none); type revolute -> fixed
- joint jRightWrist_rotz: axis 0 0 1 -> (none); limit lower=-3.14 upper=3.14 effort=200 velocity=100.0 -> (none); type revolute -> fixed

Commit message: Stabilize arm simulation and add live sensor
- Repair wrist, finger, and grasp behavior; add kinematic and physics simulation modes.
- Add live camera, EMG, and IMU feedback with recording controls inside the preview.
- Track the left arm points
mst testas

File: src/simulation/sim/arm/left_arm.urdf (robot description, URDF)
Before this commit: robot left_arm_final, 27 links, 26 joints
Links:
- link left_elbow_roty: mass 1.0 -> 0.01; geometry 
- link left_forearm: mass 0.1 -> 1.0; geometry collision mesh filename=arm/r_forearm.stl scale=-0.001 0.001 0.001; visual mesh filename=arm/r_forearm.stl scale=-0.001 0.001 0.001
- link left_hand: geometry visual mesh filename=arm/r_hand.stl scale=-0.001 0.001 0.001
- link left_wrist_rotx: geometry collision mesh filename=arm/fullhand2/LeftWristlargeV4.stl scale=0.001 0.001 0.001; visual cylinder length=0.045 radius=0.028
Joints:
- joint jLeftElbow_rotz: axis 0 0 -1 -> -1 0 0

File: src/simulation/sim/arm/right_arm.urdf (robot description, URDF)
Before this commit: robot right_arm_final, 26 links, 25 joints
Links:
- link right_wrist_rotation: geometry collision cylinder length=0.045 radius=0.028; visual cylinder length=0.045 radius=0.028

Commit message: arm flipped+ joint limit correction

File: src/simulation/sim/arm/left_arm.urdf (robot description, URDF)
Before this commit: robot left_arm_final, 27 links, 26 joints
Links:
- removed link left_elbow_roty
- removed link left_shoulder_rotx
- removed link left_wrist_rotx
- added link left_shoulder_roty, mass 0.6; collision mesh filename=arm/r_shoulder.stl scale=-0.001 0.001 0.001; collision mesh filename=arm/r_shoulder_base.stl scale=-0.001 0.001 0.001
- added link left_wrist_rotation, mass 0.1; collision cylinder length=0.045 radius=0.028; visual cylinder length=0.045 radius=0.028
- link arm_base_rotated: mass 0.001 -> 0.8
- link hand_cover_link: geometry visual mesh filename=arm/fullhand2/r_cover_hand.stl scale=-0.001 0.001 0.001
- link left_hand: mass 0.1 -> 0.4; geometry collision mesh filename=arm/r_hand.stl scale=-0.001 0.001 0.001; visual mesh filename=arm/r_hand.stl scale=-0.001 0.001 0.001
- link left_shoulder_rotz: geometry 
- link left_upper_arm: geometry collision mesh filename=arm/bicep.stl scale=-0.001 0.001 0.001; visual mesh filename=arm/bicep.stl scale=-0.001 0.001 0.001
- link thumb_link_1: geometry collision mesh filename=arm/fullhand2/r_thumb5_1.stl scale=-0.001 0.001 0.001; visual mesh filename=arm/fullhand2/r_thumb5_1.stl scale=-0.001 0.001 0.001
Joints:
- removed joint jLeftElbow_rotz
- removed joint jLeftWrist_rotx
- removed joint jLeftWrist_rotz
- added joint jLeftWrist_rotation: type revolute, parent left_forearm, child left_wrist_rotation, origin xyz=-0.310 0.0085 -0.005 rpy=0 0 0, axis 1 0 0, limit lower=0 upper=2.443461 effort=4 velocity=1.745329
- added joint left_hand_mount: type fixed, parent left_wrist_rotation, child left_hand, origin xyz=0 0 -0.006 rpy=0 0 0
- joint index_joint_1: axis 0 1 0 -> 0 -1 0
- joint index_joint_2: axis 0 1 0 -> 0 -1 0
- joint jLeftElbow_roty: child left_elbow_roty -> left_forearm; limit lower=0 upper=1.047198 effort=200 velocity=0.698132 -> lower=0 upper=1.047198 effort=10 velocity=0.698132; origin xyz=-0.305 0 0 rpy=0 0 0 -> xyz=-0.189 0 0 rpy=0 0 0
- joint jLeftShoulder_rotx: axis -1 0 0 -> 1 0 0; child left_shoulder_rotx -> left_upper_arm; limit lower=-1.047198 upper=1.047198 effort=200 velocity=0.698132 -> lower=-1.047198 upper=1.047198 effort=15 velocity=0.698132; origin xyz=0 0 0 rpy=0 0 0 -> xyz=-0.116 0 0 rpy=0 0 0; parent left_shoulder_rotz -> left_shoulder_roty
- joint jLeftShoulder_roty: axis 0 1 0 -> 0 -1 0; child left_upper_arm -> left_shoulder_roty; limit lower=0 upper=1.570796 effort=200 velocity=0.349066 -> lower=0 upper=1.308997 effort=20 velocity=0.349066; parent left_shoulder_rotx -> left_shoulder_rotz
- joint jLeftShoulder_rotz: limit lower=-0.698132 upper=-0.087266 effort=200 velocity=0.349066 -> lower=-0.698132 upper=-0.087266 effort=20 velocity=0.349066
- joint middle_joint_1: axis 0 1 0 -> 0 -1 0
- joint middle_joint_2: axis 0 1 0 -> 0 -1 0
- joint pinky_joint_1: axis 0 1 0 -> 0 -1 0
- joint pinky_joint_2: axis 0 1 0 -> 0 -1 0; origin xyz=0.003 -0.04 -0.02 rpy=-0.7 0 0 -> xyz=-0.003 -0.04 -0.02 rpy=-0.7 0 0
- joint pinky_joint_3: axis 0 1 0 -> 0 -1 0
- joint ring_joint_1: axis 0 1 0 -> 0 -1 0
- joint ring_joint_2: axis 0 1 0 -> 0 -1 0; origin xyz=0.0 -0.035 -0.017 rpy=-0.75 0 0 -> xyz=0 -0.035 -0.017 rpy=-0.75 0 0
- joint ring_joint_3: axis 0 1 0 -> 0 -1 0
- joint thumb_joint_2: origin xyz=-0.005 0.025 -0.01 rpy=2.27 0 -0.7 -> xyz=-0.005 0.025 -0.01 rpy=-2.27 0 -0.7
- joint world_to_arm_base: origin xyz=0 0 0 rpy=0 0 1.5708 -> xyz=0 0 0 rpy=0 0 -1.5708

File: src/simulation/sim/arm/right_arm.urdf (robot description, URDF)
Before this commit: robot right_arm_final, 26 links, 25 joints
Links:
- link arm_base_rotated: geometry 
- link right_shoulder_roty: geometry collision mesh filename=arm/r_shoulder.stl scale=0.001 0.001 0.001; collision mesh filename=arm/r_shoulder_base.stl scale=0.001 0.001 0.001
Joints:
- joint jRightShoulder_roty: limit lower=0 upper=1.570796 effort=20 velocity=0.349066 -> lower=0 upper=1.308997 effort=20 velocity=0.349066
