File: PCB_Designs/CAN_Transceiver/CAN_Transceiver.kicad_pcb (KiCad board)
At the start: 2 copper layers, 25 x 13 mm, 6 parts, among them J1 Conn_01x04, J2 Conn_01x02, J3 Conn_01x02, U2 SN65HVD230

Commit message: PCB Updates
Parts:
- J1: footprint Connector_PinHeader_2.54mm:PinHeader_1x04_P2.54mm_Vertical -> Connector_PinHeader_2.54mm:PinHeader_1x04_P2.54mm_Horizontal
- J2, J3: value Conn_01x02 -> CAN BUS; footprint Capacitor_THT:C_Disc_D5.0mm_W2.5mm_P2.50mm -> User_lib:J_Wurth_WR-WTB_68800211722
- moved J1 8.31 mm to (117.5, 100.0), turned to 180 degrees
- moved J2 2.75 mm to (134.0, 93.0), turned to 0 degrees
- moved J3 2.25 mm to (136.5, 98.5), turned to 180 degrees
- moved R2 1.50 mm to (130.0, 95.5)
- moved R3 1.50 mm to (128.4, 91.5)
- moved U2 1.25 mm to (125.0, 95.5)
Connections:
- J1 pad 1: +3.3V -> Net-(J1-Pin_1)
- J1 pad 2: GND -> Net-(J1-Pin_2)
- J1 pad 3: Net-(J1-Pin_3) -> GND
- J1 pad 4: Net-(J1-Pin_4) -> +3.3V
- U2 pad 1: Net-(J1-Pin_3) -> Net-(J1-Pin_1)
- U2 pad 4: Net-(J1-Pin_4) -> Net-(J1-Pin_2)
Routing:
- net Net-(J1-Pin_1): track 0.00 -> 16.6 mm
- net +3.3V: track 24.3 -> 8.08 mm
- net Net-(J1-Pin_3): track 7.16 -> 0.00 mm
- net Net-(J1-Pin_4): track 6.59 -> 0.00 mm
- net Net-(J2-Pin_1): track 18.4 -> 13.0 mm
- net Net-(J1-Pin_2): track 0.00 -> 5.06 mm
- net Net-(J2-Pin_2): track 12.4 -> 17.2 mm
