File: PCB_Designs/CAN_Transceiver/CAN_Transceiver.kicad_sch (KiCad schematic)
At the start: 6 parts, among them J1 Conn_01x04, J2 Conn_01x02, J3 Conn_01x02, U2 SN65HVD230

Commit message: PCB Updates
Parts:
- J1: footprint Connector_PinHeader_2.54mm:PinHeader_1x04_P2.54mm_Vertical -> Connector_PinHeader_2.54mm:PinHeader_1x04_P2.54mm_Horizontal
- J2, J3: value Conn_01x02 -> CAN BUS; footprint Capacitor_THT:C_Disc_D5.0mm_W2.5mm_P2.50mm -> User_lib:J_Wurth_WR-WTB_68800211722
Connections:
- net +3.3V: now also J1.4 (Pin_4); no longer J1.1 (Pin_1)
- net GND: now also J1.3 (Pin_3); no longer J1.2 (Pin_2)
- net at U2.1 (D): now also J1.1 (Pin_1); no longer J1.3 (Pin_3)
- net at U2.4 (R): now also J1.2 (Pin_2); no longer J1.4 (Pin_4)
Other:
- moved on the sheet: J1, R3
Changed lines of the file:
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@@
-	(wire
-		(pts
-			(xy 138.43 111.76) (xy 143.51 111.76)
-		)
-		(stroke
-			(width 0)
-			(type default)
-		)
-	)
-	(wire
-		(pts
-			(xy 137.16 99.06) (xy 140.97 99.06)
-		)
-		(stroke
-			(width 0)
-			(type default)
-		)
-	)
 	(wire
 		(pts
@@
 	(wire
 		(pts
-			(xy 137.16 106.68) (xy 156.21 106.68)
-		)
-		(stroke
-			(width 0)
-			(type default)
-		)
-	)
-	(wire
-		(pts
-			(xy 137.16 101.6) (xy 140.97 101.6)
-		)
-		(stroke
-			(width 0)
-			(type default)
-		)
-	)
-	(wire
-		(pts
 			(xy 204.47 113.03) (xy 204.47 114.3)
 		)
@@
 	(wire
 		(pts
+			(xy 139.7 109.22) (xy 140.97 109.22)
+		)
+		(stroke
+			(width 0)
+			(type default)
+		)
+	)
+	(wire
+		(pts
 			(xy 166.37 116.84) (xy 166.37 120.65)
 		)
@@
 	(wire
 		(pts
+			(xy 139.7 111.76) (xy 140.97 111.76)
+		)
+		(stroke
+			(width 0)
+			(type default)
+		)
+	)
+	(wire
+		(pts
 			(xy 185.42 102.87) (xy 190.5 102.87)
 		)
@@
 	(wire
 		(pts
+			(xy 151.13 119.38) (xy 151.13 124.46)
+		)
+		(stroke
+			(width 0)
+			(type default)
+		)
+	)
+	(wire
+		(pts
 			(xy 201.93 102.87) (xy 201.93 114.3)
 		)
@@
 	(wire
 		(pts
+			(xy 139.7 106.68) (xy 156.21 106.68)
+		)
+		(stroke
+			(width 0)
+			(type default)
+		)
+	)
+	(wire
+		(pts
 			(xy 190.5 113.03) (xy 204.47 113.03)
 		)
@@
 	(wire
 		(pts
-			(xy 137.16 104.14) (xy 156.21 104.14)
+			(xy 139.7 104.14) (xy 156.21 104.14)
 		)
 		(stroke
@@
 		(dnp no)
 		(property "Reference" "J2"
-			(at 204.4701 93.98 0)
+			(at 201.676 91.948 90)
 			(show_name no)
 			(do_not_autoplace no)
@@
 			)
 		)
-		(property "Value" "Conn_01x02"
-			(at 201.9301 93.98 0)
+		(property "Value" "CAN BUS"
+			(at 198.12 93.98 90)
 			(show_name no)
 			(do_not_autoplace no)
@@
 			)
 		)
-		(property "Footprint" "Capacitor_THT:C_Disc_D5.0mm_W2.5mm_P2.50mm"
+		(property "Footprint" "User_lib:J_Wurth_WR-WTB_68800211722"
 			(at 204.47 96.52 0)
 			(hide yes)
@@
 	(symbol
 		(lib_id "power:GND")
-		(at 140.97 101.6 90)
+		(at 140.97 109.22 90)
 		(unit 1)
 		(body_style 1)
@@
 		(fields_autoplaced yes)
 		(property "Reference" "#PWR03"
-			(at 147.32 101.6 0)
+			(at 147.32 109.22 0)
 			(hide yes)
 			(show_name no)
@@
 		)
 		(property "Value" "GND"
-			(at 144.78 101.5999 90)
+			(at 144.78 109.2199 90)
 			(show_name no)
 			(do_not_autoplace no)
@@
 		)
 		(property "Footprint" ""
-			(at 140.97 101.6 0)
+			(at 140.97 109.22 0)
 			(hide yes)
 			(show_name no)
@@
 		)
 		(property "Datasheet" ""
-			(at 140.97 101.6 0)
+			(at 140.97 109.22 0)
 			(hide yes)
 			(show_name no)
@@
 		)
 		(property "Description" "Power symbol creates a global label with name \"GND\" , ground"
-			(at 140.97 101.6 0)
+			(at 140.97 109.22 0)
 			(hide yes)
 			(show_name no)
@@
 	(symbol
 		(lib_id "Connector_Generic:Conn_01x04")
-		(at 132.08 101.6 0)
+		(at 134.62 106.68 0)
 		(mirror y)
 		(unit 1)
@@
 		(dnp no)
 		(property "Reference" "J1"
-			(at 132.334 96.266 0)
+			(at 134.874 101.346 0)
 			(show_name no)
 			(do_not_autoplace no)
@@
 		)
 		(property "Value" "Conn_01x04"
-			(at 132.08 110.49 0)
-			(hide yes)
-			(show_name no)
-			(do_not_autoplace no)
-			(effects
-				(font
-					(size 1.27 1.27)
-				)
-			)
-		)
-		(property "Footprint" "Connector_PinHeader_2.54mm:PinHeader_1x04_P2.54mm_Vertical"
-			(at 132.08 101.6 0)
-			(hide yes)
-			(show_name no)
-			(do_not_autoplace no)
-			(effects
-				(font
-					(size 1.27 1.27)
-				)
-			)
-		)
-		(property "Datasheet" ""
-			(at 132.08 101.6 0)
+			(at 134.62 115.57 0)
+			(hide yes)
+			(show_name no)
+			(do_not_autoplace no)
+			(effects
+				(font
+					(size 1.27 1.27)
+				)
+			)
+		)
+		(property "Footprint" "Connector_PinHeader_2.54mm:PinHeader_1x04_P2.54mm_Horizontal"
+			(at 134.62 106.68 0)
+			(hide yes)
+			(show_name no)
+			(do_not_autoplace no)
+			(effects
+				(font
+					(size 1.27 1.27)
+				)
+			)
+		)
+		(property "Datasheet" "https://www.we-online.com/components/products/datasheet/61300411021.pdf"
+			(at 134.62 106.68 0)
 			(hide yes)
 			(show_name no)
@@
 		)
 		(property "Description" "Generic connector, single row, 01x04, script generated (kicad-library-utils/schlib/autogen/connector/)"
-			(at 132.08 101.6 0)
+			(at 134.62 106.68 0)
 			(hide yes)
 			(show_name no)
@@
 	(symbol
 		(lib_id "power:+3.3V")
-		(at 140.97 99.06 270)
+		(at 140.97 111.76 270)
 		(unit 1)
 		(body_style 1)
@@
 		(fields_autoplaced yes)
 		(property "Reference" "#PWR01"
-			(at 137.16 99.06 0)
+			(at 137.16 111.76 0)
 			(hide yes)
 			(show_name no)
@@
 		)
 		(property "Value" "+3.3V"
-			(at 144.78 99.0599 90)
+			(at 144.78 111.7599 90)
 			(show_name no)
 			(do_not_autoplace no)
@@
 		)
 		(property "Footprint" ""
-			(at 140.97 99.06 0)
+			(at 140.97 111.76 0)
 			(hide yes)
 			(show_name no)
@@
 		)
 		(property "Datasheet" ""
-			(at 140.97 99.06 0)
+			(at 140.97 111.76 0)
 			(hide yes)
 			(show_name no)
@@
 		)
 		(property "Description" "Power symbol creates a global label with name \"+3.3V\""
-			(at 140.97 99.06 0)
+			(at 140.97 111.76 0)
 			(hide yes)
 			(show_name no)
@@
 	(symbol
 		(lib_id "power:GND")
-		(at 138.43 111.76 270)
+		(at 151.13 124.46 0)
 		(unit 1)
 		(body_style 1)
@@
 		(fields_autoplaced yes)
 		(property "Reference" "#PWR05"
-			(at 132.08 111.76 0)
+			(at 151.13 130.81 0)
 			(hide yes)
 			(show_name no)
@@
 		)
 		(property "Value" "GND"
-			(at 134.62 111.7599 90)
-			(show_name no)
-			(do_not_autoplace no)
-			(effects
-				(font
-					(size 1.27 1.27)
-				)
-				(justify right)
+			(at 153.67 125.7299 0)
+			(show_name no)
+			(do_not_autoplace no)
+			(effects
+				(font
+					(size 1.27 1.27)
+				)
+				(justify left)
 			)
 		)
 		(property "Footprint" ""
-			(at 138.43 111.76 0)
+			(at 151.13 124.46 0)
 			(hide yes)
 			(show_name no)
@@
 		)
 		(property "Datasheet" ""
-			(at 138.43 111.76 0)
+			(at 151.13 124.46 0)
 			(hide yes)
 			(show_name no)
@@
 		)
 		(property "Description" "Power symbol creates a global label with name \"GND\" , ground"
-			(at 138.43 111.76 0)
+			(at 151.13 124.46 0)
 			(hide yes)
 			(show_name no)
@@
 	(symbol
 		(lib_id "Device:R")
-		(at 147.32 111.76 270)
+		(at 151.13 115.57 0)
 		(unit 1)
 		(body_style 1)
@@
 		(dnp no)
 		(property "Reference" "R3"
-			(at 146.558 114.554 90)
+			(at 153.924 116.332 90)
 			(show_name no)
 			(do_not_autoplace no)
@@
 		)
 		(property "Value" "10kOhm"
-			(at 147.32 108.712 90)
+			(at 148.082 115.57 90)
 			(show_name no)
 			(do_not_autoplace no)
@@
 		)
 		(property "Footprint" "Resistor_SMD:R_0603_1608Metric_Pad0.98x0.95mm_HandSolder"
-			(at 147.32 109.982 90)
+			(at 149.352 115.57 90)
 			(hide yes)
 			(show_name no)
@@
 		)
 		(property "Datasheet" ""
-			(at 147.32 111.76 0)
+			(at 151.13 115.57 0)
 			(hide yes)
 			(show_name no)
@@
 		)
 		(property "Description" "Resistor"
-			(at 147.32 111.76 0)
+			(at 151.13 115.57 0)
 			(hide yes)
 			(show_name no)
@@
 		(dnp no)
 		(property "Reference" "J3"
-			(at 201.9299 121.92 0)
+			(at 203.962 122.174 90)
 			(show_name no)
 			(do_not_autoplace no)
@@
 			)
 		)
-		(property "Value" "Conn_01x02"
-			(at 204.4699 121.92 0)
+		(property "Value" "CAN BUS"
+			(at 207.772 123.952 90)
 			(show_name no)
 			(do_not_autoplace no)
@@
 			)
 		)
-		(property "Footprint" "Capacitor_THT:C_Disc_D5.0mm_W2.5mm_P2.50mm"
+		(property "Footprint" "User_lib:J_Wurth_WR-WTB_68800211722"
 			(at 201.93 119.38 0)
 			(hide yes)
@@
 			)
 		)
-		(property "Datasheet" ""
+		(property "Datasheet" "https://www.we-online.com/en/components/products/WTB_WR_WTB_2_50_MM_J_MALE#/articles/WTB_WR_WTB_2_50_MM_MALE_J_HORIZONTAL"
 			(at 201.93 119.38 0)
 			(hide yes)
@@
 		(dnp no)
 		(property "Reference" "R2"
-			(at 185.166 114.3 0)
+			(at 192.024 106.172 0)
 			(show_name no)
 			(do_not_autoplace no)
@@
 		)
 		(property "Value" "120 Ohm"
-			(at 187.96 114.3 0)
-			(show_name no)
-			(do_not_autoplace no)
+			(at 192.024 108.204 0)
+			(show_name no)
+			(do_not_autoplace no)
