File: PCB_Designs/Hand_Motor/Hand_Motor.kicad_pcb (KiCad board)
At the start: 2 copper layers, 74 x 31 mm, 9 parts, among them J1 Power In, J12 68800611722, J14 613004143121: CAN-BUS, J2 IMU, U1 ESP32-C3-Zero

Commit message: PCB Updates
Parts:
- J1: footprint Connector_THT_Wurth:J_Wurth_WR-NPC2_626002110201 -> User_lib:J_Wurth_WR-NPC2_626002110201
- J12: footprint Connector_THT_Wurth:J_Wurth_WR-WTB_68800611722 -> User_lib:J_Wurth_WR-WTB_68800611722
- J2: footprint Connector_THT_Wurth:J_Wurth_WR-WTB_68800411622 -> User_lib:J_Wurth_WR-WTB_68800411622
