File: PCB_Designs/Hand_Pressure/Hand_Pressure.kicad_pcb (KiCad board)
At the start: 2 copper layers, 71 x 31.1 mm, 13 parts, among them J1 Power In, J2 IMU, J4 61301021121, J5 IMU, U1 ESP32-C3-Zero

Commit message: PCB Updates
Parts:
- J1: footprint Connector_THT_Wurth:J_Wurth_WR-NPC2_626002110201 -> User_lib:J_Wurth_WR-NPC2_626002110201
- J2: footprint Connector_THT_Wurth:J_Wurth_WR-WTB_68800411622 -> User_lib:J_Wurth_WR-WTB_68800411622
- J4: footprint Connector_THT_Wurth:J_Wurth_WR-PHD_61301021121 -> User_lib:J_Wurth_WR-PHD_61301021121
